File: SmartParallel.sch (KiCad schematic (older format))
At the start: 47 parts, among them IC1 S74HC595, J1 DB25, P1 SERIAL_PORT, P2 PWR_IN, P3 PWR_OUT, P4 PWR_OUT, P5 I2C_DISPLAY, P6 REM_RESET, SW2 SW_RST, U1 ATMEGA328PB, U2 74HC541, U3 74HC14MS, Y1 16MHz

Commit message: Fixed library issues
Parts:
- D1, D2, D3, D4, D5, D6, D7: symbol SmartParallel-rescue:Led_Small -> Device:LED_Small
- J1: symbol SmartParallel-rescue:DB25 -> speculatrix_connectors:DB25
- P1: symbol SmartParallel-rescue:CONN_01X06 -> Connector:Conn_01x06_Male
- P2, P3, P4, P6: symbol SmartParallel-rescue:CONN_01X02 -> Connector:Conn_01x02_Male
- P5: symbol SmartParallel-rescue:CONN_01X04 -> Connector:Conn_01x04_Male
- U2: symbol SmartParallel-rescue:74HC541-speculatrix_ic -> speculatrix_ic:74HC541
Connections:
- net CTS: now also P1.2 (Pin_2); no longer P1.5 (P5)
- net GND: now also P1.1 (Pin_1), P2.1 (Pin_1), P3.1 (Pin_1), P4.1 (Pin_1), P5.1 (Pin_1), P6.1 (Pin_1), U2.19 (~OE2); no longer P1.6 (P6), P2.2 (P2), P3.2 (P2), P4.2 (P2), P5.4 (P4), P6.2 (P2), U2.~ (~OE2)
- net RTS: now also P1.6 (Pin_6); no longer P1.1 (P1)
- net RXD: now also P1.4 (Pin_4); no longer P1.3 (P3)
- net SCL: now also P5.2 (Pin_2); no longer P5.3 (P3)
- net SDA: now also P5.3 (Pin_3); no longer P5.2 (P2)
- net TXD: now also P1.5 (Pin_5); no longer P1.2 (P2)
- net VCC: now also P1.3 (Pin_3), P2.2 (Pin_2), P3.2 (Pin_2), P4.2 (Pin_2), P5.4 (Pin_4); no longer P1.4 (P4), P2.1 (P1), P3.1 (P1), P4.1 (P1), P5.1 (P1)
- net ~RESET: now also P6.2 (Pin_2); no longer P6.1 (P1)
Changed lines of the file:
@@
 $EndComp
 $Comp
-L SmartParallel-rescue:DB25 J1
+L speculatrix_connectors:DB25 J1
 U 1 1 5AB65516
 P 10850 3600
@@
 Text GLabel 4250 3000 2    50   Input ~ 0
 ~RESET
-$Comp
-L SmartParallel-rescue:CONN_01X06 P1
-U 1 1 5AB667A6
-P 1175 6850
-F 0 "P1" H 1175 7200 50  0000 C CNN
-F 1 "SERIAL_PORT" V 1275 6850 50  0000 C CNN
-F 2 "Pin_Headers:Pin_Header_Straight_1x06" H 1175 6850 50  0001 C CNN
-F 3 "" H 1175 6850 50  0000 C CNN
-	1    1175 6850
-	-1   0    0    1
-$EndComp
 Text GLabel 1375 6900 2    50   Input ~ 0
 RXD
 $Comp
-L SmartParallel-rescue:CONN_01X02 P2
+L Connector:Conn_01x02_Male P2
 U 1 1 5AB668DC
-P 2150 1175
-F 0 "P2" H 2150 1325 50  0000 C CNN
-F 1 "PWR_IN" V 2250 1175 50  0000 C CNN
-F 2 "Pin_Headers:Pin_Header_Straight_1x02" H 2150 1175 50  0001 C CNN
-F 3 "" H 2150 1175 50  0000 C CNN
-	1    2150 1175
-	1    0    0    -1
+P 2150 1225
+F 0 "P2" H 2175 1000 50  0000 C CNN
+F 1 "PWR_IN" V 2075 1175 50  0000 C CNN
+F 2 "Pin_Headers:Pin_Header_Straight_1x02" H 2150 1225 50  0001 C CNN
+F 3 "" H 2150 1225 50  0000 C CNN
+	1    2150 1225
+	-1   0    0    1
 $EndComp
 $Comp
@@
 ~RESET
 $Comp
-L SmartParallel-rescue:Led_Small D3
+L Device:LED_Small D3
 U 1 1 5AB69C3C
 P 4450 4600
@@
 $EndComp
 $Comp
-L SmartParallel-rescue:Led_Small D2
+L Device:LED_Small D2
 U 1 1 5AB69D3C
 P 4750 4600
@@
 $EndComp
 $Comp
-L SmartParallel-rescue:74HC541-speculatrix_ic U2
+L speculatrix_ic:74HC541 U2
 U 1 1 5AB76375
 P 6500 5200
@@
 $EndComp
 $Comp
-L SmartParallel-rescue:Led_Small D1
+L Device:LED_Small D1
 U 1 1 5AB788F6
 P 5050 4600
@@
 $EndComp
 $Comp
-L SmartParallel-rescue:CONN_01X04 P5
+L Connector:Conn_01x04_Male P5
 U 1 1 5AD5CFB3
-P 3675 7050
-F 0 "P5" H 3675 7300 50  0000 C CNN
-F 1 "I2C_DISPLAY" V 3775 7050 50  0000 C CNN
-F 2 "Pin_Headers:Pin_Header_Straight_1x04" H 3675 7050 50  0001 C CNN
-F 3 "" H 3675 7050 50  0000 C CNN
-	1    3675 7050
-	1    0    0    -1
+P 3675 7100
+F 0 "P5" H 3775 7350 50  0000 C CNN
+F 1 "I2C_DISPLAY" V 3550 7100 50  0000 C CNN
+F 2 "Pin_Headers:Pin_Header_Straight_1x04" H 3675 7100 50  0001 C CNN
+F 3 "" H 3675 7100 50  0000 C CNN
+	1    3675 7100
+	-1   0    0    1
 $EndComp
 Text GLabel 3475 7000 0    50   Input ~ 0
@@
 	1300 1375 1300 1475
 Wire Wire Line
-	1950 925  1950 1125
-Wire Wire Line
 	1300 775  1300 925
 Wire Wire Line
@@
 Connection ~ 1700 1375
 $Comp
-L SmartParallel-rescue:CONN_01X02 P6
+L Connector:Conn_01x02_Male P6
 U 1 1 5AD8D38D
-P 6300 750
-F 0 "P6" H 6300 900 50  0000 C CNN
-F 1 "REM_RESET" V 6400 750 50  0000 C CNN
-F 2 "Pin_Headers:Pin_Header_Straight_1x02" H 6300 750 50  0001 C CNN
-F 3 "" H 6300 750 50  0000 C CNN
-	1    6300 750
-	1    0    0    -1
+P 6300 800
+F 0 "P6" H 6375 575 50  0000 C CNN
+F 1 "REM_RESET" V 6200 750 50  0000 C CNN
+F 2 "Pin_Headers:Pin_Header_Straight_1x02" H 6300 800 50  0001 C CNN
+F 3 "" H 6300 800 50  0000 C CNN
+	1    6300 800
+	-1   0    0    1
 $EndComp
 Wire Wire Line
@@
 Connection ~ 5450 1850
 $Comp
-L SmartParallel-rescue:CONN_01X02 P3
+L Connector:Conn_01x02_Male P3
 U 1 1 5AEAF775
-P 2650 1175
-F 0 "P3" H 2650 1325 50  0000 C CNN
-F 1 "PWR_OUT" V 2750 1175 50  0000 C CNN
-F 2 "Pin_Headers:Pin_Header_Straight_1x02" H 2650 1175 50  0001 C CNN
-F 3 "" H 2650 1175 50  0000 C CNN
-	1    2650 1175
-	1    0    0    -1
-$EndComp
-$Comp
-L SmartParallel-rescue:CONN_01X02 P4
+P 2650 1225
+F 0 "P3" H 2750 1000 50  0000 C CNN
+F 1 "PWR_OUT" V 2525 1175 50  0000 C CNN
+F 2 "Pin_Headers:Pin_Header_Straight_1x02" H 2650 1225 50  0001 C CNN
+F 3 "" H 2650 1225 50  0000 C CNN
+	1    2650 1225
+	-1   0    0    1
+$EndComp
+$Comp
+L Connector:Conn_01x02_Male P4
 U 1 1 5AEAF7D8
-P 3300 1175
-F 0 "P4" H 3300 1325 50  0000 C CNN
-F 1 "PWR_OUT" V 3400 1175 50  0000 C CNN
-F 2 "Pin_Headers:Pin_Header_Straight_1x02" H 3300 1175 50  0001 C CNN
-F 3 "" H 3300 1175 50  0000 C CNN
-	1    3300 1175
-	1    0    0    -1
-$EndComp
-Wire Wire Line
-	2450 925  2450 1125
+P 3300 1225
+F 0 "P4" H 3400 1000 50  0000 C CNN
+F 1 "PWR_OUT" V 3225 1175 50  0000 C CNN
+F 2 "Pin_Headers:Pin_Header_Straight_1x02" H 3300 1225 50  0001 C CNN
+F 3 "" H 3300 1225 50  0000 C CNN
+	1    3300 1225
+	-1   0    0    1
+$EndComp
 Connection ~ 1950 925
-Wire Wire Line
-	3100 925  3100 1125
 Connection ~ 2450 925
 Wire Wire Line
 	2450 1375 2450 1225
-Connection ~ 1950 1375
 Wire Wire Line
 	3100 1375 3100 1225
-Connection ~ 2450 1375
 Text GLabel 9025 800  1    50   Input ~ 0
 D0
@@
 $EndComp
 $Comp
-L SmartParallel-rescue:Led_Small D4
+L Device:LED_Small D4
 U 1 1 5B05F13A
 P 8450 5500
@@
 $EndComp
 $Comp
-L SmartParallel-rescue:Led_Small D5
+L Device:LED_Small D5
 U 1 1 5B060918
 P 8650 5500
@@
 $EndComp
 $Comp
-L SmartParallel-rescue:Led_Small D6
+L Device:LED_Small D6
 U 1 1 5B0609D2
 P 8850 5500
@@
 $EndComp
 $Comp
-L SmartParallel-rescue:Led_Small D7
+L Device:LED_Small D7
 U 1 1 5B06104A
 P 9050 5500
@@
 Wire Wire Line
 	2450 925  3100 925
-Wire Wire Line
-	1950 1375 2450 1375
-Wire Wire Line
-	2450 1375 3100 1375
 Wire Wire Line
 	5650 4900 6050 4900
@@
 	2550 4050 2350 4050
 Connection ~ 2350 4050
+$Comp
+L Connector:Conn_01x06_Male P1
+U 1 1 5AB667A6
+P 1175 6800
+F 0 "P1" H 1450 7100 50  0000 C CNN
+F 1 "SERIAL_PORT" V 1075 6750 50  0000 C CNN
+F 2 "Pin_Headers:Pin_Header_Straight_1x06" H 1175 6800 50  0001 C CNN
+F 3 "" H 1175 6800 50  0000 C CNN
+	1    1175 6800
+	1    0    0    -1
+$EndComp
+Wire Wire Line
+	1950 1375 2450 1375
+Wire Wire Line
+	1950 925  1950 1125
+Connection ~ 1950 1375
+Wire Wire Line
+	2450 925  2450 1125
+Wire Wire Line
+	3100 1375 2450 1375
+Wire Wire Line
+	3100 925  3100 1125
+Connection ~ 2450 1375
 $EndSCHEMATC

Commit message: Minor updates
Parts:
- CONN1: footprint speculatrix_connectors:AVR_ISP_HE10_2x3 -> Speculatrix_connectors:AVR_ISP_HE10_2x3
Changed lines of the file:
@@
 F 0 "CONN1" H 5525 7300 60  0000 C CNN
 F 1 "AVR-ISP" H 5525 6650 60  0000 C CNN
-F 2 "speculatrix_connectors:AVR_ISP_HE10_2x3" H 5725 6850 60  0001 C CNN
+F 2 "Speculatrix_connectors:AVR_ISP_HE10_2x3" H 5725 6850 60  0001 C CNN
 F 3 "" H 5725 6850 60  0000 C CNN
 	1    5525 7000

Commit message: First completed PCB
Connections:
- net Busy: now also U2.5 (A4); no longer U2.4 (A3)
- net Busy_buf: now also U1.22 ((MOSI1)_PE3), U2.15 (Y4); no longer U1.2 (PD4), U2.16 (Y3)
- net CTS: now also U1.2 (PD4); no longer U1.11 (PD7)
- net PE: now also U2.3 (A2); no longer U2.6 (A5)
- net PE_buf: now also U1.6 ((SCL1)_PE1), U2.17 (Y2); no longer U1.10 (PD6), U2.14 (Y5)
- net RTS: now also U1.1 (PD3); no longer U1.3 ((SDA1)_PE0)
- net SEL: now also U2.4 (A3); no longer U2.5 (A4)
- net Sel_buf: now also U1.19 (PE2), U2.16 (Y3); no longer U1.9 (PD5), U2.15 (Y4)
- net ~Error: now also U2.6 (A5); no longer U2.3 (A2)
- net Stat2: now reaches D2.2 (A)
- net Stat2: now also U1.10 (PD6); no longer U1.19 (PE2)
- net Stat3: now reaches D3.2 (A)
- net Stat3: now also U1.11 (PD7); no longer U1.22 ((MOSI1)_PE3)
- net Stat1: now reaches D1.2 (A)
- net Stat1: now also U1.9 (PD5); no longer U1.6 ((SCL1)_PE1)
- net XTAL1: now reaches C4.1, U1.7 (PB6_(XTAL1)), Y1.1
- net XTAL2: now reaches C5.1, U1.8 (PB7_(XTAL2)), Y1.2
- removed net Error_buf: U1.1 (PD3), U2.17 (Y2)
- new net Err_buf: U1.3 ((SDA1)_PE0), U2.14 (Y5)
Other:
- note added: "328PB -> Signal buffer\nAck_buf\nErr_buf\nPE_buf\nSel_buf\nBusy_buf"
- moved on the sheet: D1, D2, D3, R3, R6, R8
Changed lines of the file:
@@
 Sheet 1 1
 Title "SmartParallel"
-Date "2019-05-21"
+Date "2019-06-06"
 Rev "1.0"
 Comp "Machina Speculatrix"
@@
 L power:GND #PWR05
 U 1 1 5AB673B3
-P 1500 5450
-F 0 "#PWR05" H 1500 5200 50  0001 C CNN
-F 1 "GND" H 1500 5300 50  0000 C CNN
-F 2 "" H 1500 5450 50  0000 C CNN
-F 3 "" H 1500 5450 50  0000 C CNN
-	1    1500 5450
+P 1500 4500
+F 0 "#PWR05" H 1500 4250 50  0001 C CNN
+F 1 "GND" H 1500 4350 50  0000 C CNN
+F 2 "" H 1500 4500 50  0000 C CNN
+F 3 "" H 1500 4500 50  0000 C CNN
+	1    1500 4500
 	1    0    0    -1
 $EndComp
@@
 Text GLabel 4250 3150 2    50   Input ~ 0
 RXD
-Text GLabel 6050 4800 0    50   Input ~ 0
+Text GLabel 6050 4900 0    50   Input ~ 0
 Busy
 Text GLabel 5050 2600 2    50   Input ~ 0
 LF
-Text GLabel 5550 4700 0    50   Input ~ 0
+Text GLabel 5475 5000 0    50   Input ~ 0
 ~Error
 Text GLabel 5550 4600 0    50   Input ~ 0
@@
 Text GLabel 5050 2700 2    50   Input ~ 0
 ~SelIn
-Text GLabel 5500 4900 0    50   Input ~ 0
+Text GLabel 5500 4800 0    50   Input ~ 0
 SEL
-Text GLabel 6050 5000 0    50   Input ~ 0
+Text GLabel 6050 4700 0    50   Input ~ 0
 PE
 NoConn ~ 9250 2650
@@
 L Device:LED_Small D3
 U 1 1 5AB69C3C
-P 4450 4600
-F 0 "D3" H 4400 4725 50  0000 L CNN
-F 1 "STAT3" H 4275 4500 50  0000 L CNN
-F 2 "LEDs:LED_1206" V 4450 4600 50  0001 C CNN
-F 3 "" V 4450 4600 50  0000 C CNN
-	1    4450 4600
+P 4225 5175
+F 0 "D3" H 4175 5300 50  0000 L CNN
+F 1 "STAT3" H 4050 5075 50  0000 L CNN
+F 2 "LEDs:LED_1206" V 4225 5175 50  0001 C CNN
+F 3 "" V 4225 5175 50  0000 C CNN
+	1    4225 5175
 	0    -1   -1   0
 $EndComp
@@
 L Device:R R3
 U 1 1 5AB69CAB
-P 4450 4950
-F 0 "R3" V 4530 4950 50  0000 C CNN
-F 1 "330" V 4450 4950 50  0000 C CNN
-F 2 "Resistors_SMD:R_1206" V 4380 4950 50  0001 C CNN
-F 3 "" H 4450 4950 50  0000 C CNN
-	1    4450 4950
+P 4225 5525
+F 0 "R3" V 4305 5525 50  0000 C CNN
+F 1 "330" V 4225 5525 50  0000 C CNN
+F 2 "Resistors_SMD:R_1206" V 4155 5525 50  0001 C CNN
+F 3 "" H 4225 5525 50  0000 C CNN
+	1    4225 5525
 	1    0    0    -1
 $EndComp
@@
 L Device:R R6
 U 1 1 5AB69CEA
-P 4750 4950
-F 0 "R6" V 4830 4950 50  0000 C CNN
-F 1 "330" V 4750 4950 50  0000 C CNN
-F 2 "Resistors_SMD:R_1206" V 4680 4950 50  0001 C CNN
-F 3 "" H 4750 4950 50  0000 C CNN
-	1    4750 4950
+P 4525 5525
+F 0 "R6" V 4605 5525 50  0000 C CNN
+F 1 "330" V 4525 5525 50  0000 C CNN
+F 2 "Resistors_SMD:R_1206" V 4455 5525 50  0001 C CNN
+F 3 "" H 4525 5525 50  0000 C CNN
+	1    4525 5525
 	1    0    0    -1
 $EndComp
@@
 L Device:LED_Small D2
 U 1 1 5AB69D3C
-P 4750 4600
-F 0 "D2" H 4700 4725 50  0000 L CNN
-F 1 "STAT2" H 4575 4500 50  0000 L CNN
-F 2 "LEDs:LED_1206" V 4750 4600 50  0001 C CNN
-F 3 "" V 4750 4600 50  0000 C CNN
-	1    4750 4600
+P 4525 5175
+F 0 "D2" H 4475 5300 50  0000 L CNN
+F 1 "STAT2" H 4350 5075 50  0000 L CNN
+F 2 "LEDs:LED_1206" V 4525 5175 50  0001 C CNN
+F 3 "" V 4525 5175 50  0000 C CNN
+	1    4525 5175
 	0    -1   -1   0
 $EndComp
@@
 	1    0    0    -1
 $EndComp
-Text Label 4900 3350 2    60   ~ 0
-Ack_buf
-Text Label 4900 3550 2    60   ~ 0
-Busy_buf
-Text Label 4950 3450 2    60   ~ 0
-Error_buf
-Text Label 4850 3650 2    60   ~ 0
-Sel_buf
-Text Label 4850 3750 2    60   ~ 0
-PE_buf
 Text GLabel 10400 4800 0    50   Input ~ 0
 Strobe_buf
@@
 L Device:R R8
 U 1 1 5AB78890
-P 5050 4950
-F 0 "R8" V 5130 4950 50  0000 C CNN
-F 1 "330" V 5050 4950 50  0000 C CNN
-F 2 "Resistors_SMD:R_1206" V 4980 4950 50  0001 C CNN
-F 3 "" H 5050 4950 50  0000 C CNN
-	1    5050 4950
+P 4825 5525
+F 0 "R8" V 4905 5525 50  0000 C CNN
+F 1 "330" V 4825 5525 50  0000 C CNN
+F 2 "Resistors_SMD:R_1206" V 4755 5525 50  0001 C CNN
+F 3 "" H 4825 5525 50  0000 C CNN
+	1    4825 5525
 	1    0    0    -1
 $EndComp
@@
 L Device:LED_Small D1
 U 1 1 5AB788F6
-P 5050 4600
-F 0 "D1" H 5000 4725 50  0000 L CNN
-F 1 "STAT1" H 4875 4500 50  0000 L CNN
-F 2 "LEDs:LED_1206" V 5050 4600 50  0001 C CNN
-F 3 "" V 5050 4600 50  0000 C CNN
-	1    5050 4600
+P 4825 5175
+F 0 "D1" H 4775 5300 50  0000 L CNN
+F 1 "STAT1" H 4650 5075 50  0000 L CNN
+F 2 "LEDs:LED_1206" V 4825 5175 50  0001 C CNN
+F 3 "" V 4825 5175 50  0000 C CNN
+	1    4825 5175
 	0    -1   -1   0
 $EndComp
@@
 	4550 1150 4750 1150
 Wire Wire Line
-	4250 4300 4450 4300
-Wire Wire Line
-	4450 4300 4450 4500
-Wire Wire Line
-	4250 4200 4750 4200
-Wire Wire Line
-	4750 4200 4750 4500
-Wire Wire Line
-	4750 4700 4750 4800
-Wire Wire Line
-	4450 4700 4450 4800
-Wire Wire Line
-	4450 5100 4450 5200
-Wire Wire Line
-	1500 5200 4450 5200
-Wire Wire Line
-	4750 5200 4750 5100
-Connection ~ 4450 5200
+	4525 5275 4525 5375
+Wire Wire Line
+	4225 5275 4225 5375
+Wire Wire Line
+	4225 5675 4225 5775
+Wire Wire Line
+	4525 5775 4525 5675
 Wire Wire Line
 	5850 3950 5850 4050
@@
 Connection ~ 5850 4050
 Wire Wire Line
-	6900 4600 7000 4600
-Wire Wire Line
-	7000 4600 7000 3350
-Wire Wire Line
-	7000 3350 4250 3350
-Wire Wire Line
-	6900 4700 7050 4700
-Wire Wire Line
-	7050 4700 7050 3450
-Wire Wire Line
-	7050 3450 4250 3450
-Wire Wire Line
-	6900 4800 7100 4800
-Wire Wire Line
-	7100 4800 7100 3550
-Wire Wire Line
-	7100 3550 4250 3550
-Wire Wire Line
-	6900 4900 7150 4900
-Wire Wire Line
-	7150 4900 7150 3650
-Wire Wire Line
-	7150 3650 4250 3650
-Wire Wire Line
-	6900 5000 7200 5000
-Wire Wire Line
-	7200 5000 7200 3750
-Wire Wire Line
-	7200 3750 4250 3750
-Wire Wire Line
 	4750 1100 4750 1150
 Connection ~ 4750 1150
 Wire Wire Line
-	4250 4100 5050 4100
-Wire Wire Line
-	5050 4100 5050 4500
-Wire Wire Line
-	5050 4700 5050 4800
-Wire Wire Line
-	5050 5200 5050 5100
-Connection ~ 4750 5200
+	4825 5275 4825 5375
+Wire Wire Line
+	4825 5775 4825 5675
+Connection ~ 4525 5775
 Wire Wire Line
 	4250 2500 4700 2500
@@
 Wire Wire Line
 	6100 700  4950 700
-Text GLabel 4250 3850 2    50   Input ~ 0
+Text GLabel 4250 3550 2    50   Input ~ 0
 CTS
 Text GLabel 1375 6700 2    50   Input ~ 0
 CTS
-Text GLabel 4250 4000 2    50   Input ~ 0
+Text GLabel 4250 3450 2    50   Input ~ 0
 RTS
 Text GLabel 1375 7100 2    50   Input ~ 0
@@
 Wire Wire Line
 	6075 7200 5975 7200
-Wire Wire Line
-	5550 4700 5700 4700
-Wire Wire Line
-	5700 4400 5700 4700
-Connection ~ 5700 4700
 Wire Wire Line
 	4700 1850 4800 1850
@@
 $EndComp
 Wire Wire Line
-	5500 4900 5650 4900
-Wire Wire Line
-	5650 5050 5650 4900
-Connection ~ 5650 4900
-Wire Wire Line
 	5650 5350 5650 5650
 $Comp
@@
 	4900 2400 5050 2400
 Wire Wire Line
-	1500 5200 1500 5450
-Wire Wire Line
-	4450 5200 4750 5200
+	4225 5775 4525 5775
 Wire Wire Line
 	5850 5400 6050 5400
@@
 	4750 1150 4950 1150
 Wire Wire Line
-	4750 5200 5050 5200
+	4525 5775 4825 5775
 Wire Wire Line
 	4700 2500 5050 2500
@@
 	1700 1375 1950 1375
 Wire Wire Line
-	5700 4700 6050 4700
-Wire Wire Line
 	4800 1850 4900 1850
 Wire Wire Line
@@
 Wire Wire Line
 	2450 925  3100 925
-Wire Wire Line
-	5650 4900 6050 4900
 Wire Wire Line
 	9400 6125 9400 6350
@@
 Wire Wire Line
 	1500 4050 1500 4300
-Connection ~ 1500 5200
 Connection ~ 1500 4300
-Wire Wire Line
-	1500 4300 1500 5200
 Wire Wire Line
 	1500 2900 1500 2500
@@
 	3100 925  3100 1125
 Connection ~ 2450 1375
+Text Label 2400 3700 0    50   ~ 0
+XTAL1
+Text Label 2625 3800 0    50   ~ 0
+XTAL2
+Text GLabel 4250 3350 2    50   Input ~ 0
+Ack_buf
+Text GLabel 6900 4600 2    50   Input ~ 0
+Ack_buf
+Text GLabel 4250 4000 2    50   Input ~ 0
+Err_buf
+Text GLabel 6900 5000 2    50   Input ~ 0
+Err_buf
+Text GLabel 4250 4300 2    50   Input ~ 0
+Busy_buf
+Text GLabel 6900 4900 2    50   Input ~ 0
+Busy_buf
+Text GLabel 4250 4200 2    50   Input ~ 0
+Sel_buf
+Text GLabel 6900 4800 2    50   Input ~ 0
+Sel_buf
+Text GLabel 4250 4100 2    50   Input ~ 0
+PE_buf
+Text GLabel 6900 4700 2    50   Input ~ 0
+PE_buf
+Text GLabel 4250 3750 2    50   Input ~ 0
+Stat2
+Text GLabel 4525 5075 1    50   Input ~ 0
+Stat2
+Text GLabel 4250 3650 2    50   Input ~ 0
+Stat1
+Text GLabel 4250 3850 2    50   Input ~ 0
+Stat3
+Text GLabel 4825 5075 1    50   Input ~ 0
+Stat1
+Wire Wire Line
+	1500 4300 1500 4500
+$Comp
+L power:GND #PWR0102
+U 1 1 5CFA0836
+P 4525 5950
+F 0 "#PWR0102" H 4525 5700 50  0001 C CNN
+F 1 "GND" H 4525 5800 50  0000 C CNN
+F 2 "" H 4525 5950 50  0000 C CNN
+F 3 "" H 4525 5950 50  0000 C CNN
+	1    4525 5950
+	1    0    0    -1
+$EndComp
+Wire Wire Line
+	4525 5950 4525 5775
+Text GLabel 4225 5075 1    50   Input ~ 0
+Stat3
+Text Notes 1075 5375 0    50   ~ 0
+328PB -> Signal buffer\nAck_buf\nErr_buf\nPE_buf\nSel_buf\nBusy_buf
+Wire Wire Line
+	5475 5000 5700 5000
+Wire Wire Line
+	5700 4400 5700 5000
+Connection ~ 5700 5000
+Wire Wire Line
+	5700 5000 6050 5000
+Wire Wire Line
+	5500 4800 5650 4800
+Wire Wire Line
+	5650 5050 5650 4800
+Connection ~ 5650 4800
+Wire Wire Line
+	5650 4800 6050 4800
 $EndSCHEMATC

Commit message: minor update
Other:
- note removed: "328PB -> Signal buffer\nAck_buf\nErr_buf\nPE_buf\nSel_buf\nBusy_buf"
Changed lines of the file:
@@
 Text GLabel 4225 5075 1    50   Input ~ 0
 Stat3
-Text Notes 1075 5375 0    50   ~ 0
-328PB -> Signal buffer\nAck_buf\nErr_buf\nPE_buf\nSel_buf\nBusy_buf
 Wire Wire Line
 	5475 5000 5700 5000

Commit message: many small changes
Parts:
- removed LED1: BAR_LED8, Speculatrix_general:8-bar LED, symbol speculatrix_display:BAR_LED8
- removed RN1: 580, Resistors_ThroughHole:Resistor_Array_SIP8, symbol Device:R_Network08
- added C9: 1µF, Capacitors_SMD:C_1206, symbol Device:C
- added D8, D9: D, symbol Device:D
- added R1: 330, Resistors_SMD:R_1206, symbol Device:R
- added R2: 10K, Resistors_SMD:R_1206, symbol Device:R
- D4: value Strobe -> Autofeed
- R15: value 470 -> 10K
- R16, R17, R18: value 470 -> 330
- R4: value 10K -> 1K
Connections:
- net Busy: no longer D7.2 (A)
- net Busy_buf: now also D7.2 (A)
- net GND: now also C9.2, R1.2; no longer R11.2
- net RTS: now also U1.3 ((SDA1)_PE0); no longer U1.1 (PD3)
- net SEL: now also R11.2, U3.3 (2A); no longer R11.1, U3.5 (3A)
- net VCC: now also U3.11 (5A), U3.13 (6A), U3.9 (4A), C9.1, D8.2 (A), D9.2 (A); no longer R10.1, R12.1, R13.1, R4.1, R7.1, R9.1
- net ~Error: now also U3.1 (1A); no longer U3.3 (2A)
- net at D4.1 (K): now also R1.1; no longer R15.1
- net at U3.2 (1Y): now also D5.2 (A); no longer D4.2 (A)
- net at U3.4 (2Y): now also D6.2 (A); no longer D5.2 (A)
- net at U3.6 (3Y): now also D4.2 (A); no longer D6.2 (A)
- net Ack_buf renamed ~Ack_buf
- net Err_buf renamed ~Err_buf
- net ~Err_buf: now also U1.1 (PD3); no longer U1.3 ((SDA1)_PE0)
- net Init_buf renamed ~Init_buf
- net LF renamed ~Autofeed
- net ~Autofeed: now also R2.2
- net LF_buf renamed ~Autofeed_buf
- net ~Autofeed_buf: now also U3.5 (3A)
- net Strobe_buf renamed ~Strobe_buf
- net ~Strobe_buf: no longer U3.1 (1A)
- net ~SelIn renamed SelIn
- net SelIn: now also R15.1
- new net: D9.1 (K), R11.1, R12.1, R13.1
- new net: D8.1 (K), R10.1, R2.1, R4.1, R7.1, R9.1
- no-connect marks 8 -> 6
Other:
- note removed: "Data Blinkenlights"
- moved on the sheet: C6, C7, D1, D2, D3, D5, D6, D7, IC1, R11, R12, R13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

Commit message: Final version of Rev.2.0 schematic
Parts:
- removed IC1: S74HC595, Housings_SOIC:SOIC-16_3.9x9.9mm_Pitch1.27mm, symbol speculatrix_ic:S74HC595
- removed P4: PWR_OUT, Pin_Headers:Pin_Header_Straight_1x02, symbol Connector:Conn_01x02_Male
- removed U2: 74HC541, Housings_SOIC:SOIC-20W_7.5x12.8mm_Pitch1.27mm, symbol speculatrix_ic:74HC541
- removed U3: 74HC14MS, Housings_SOIC:SOIC-14_3.9x8.7mm_Pitch1.27mm, symbol speculatrix_ic:74HC14MS
- added D3: PWR, LEDs:LED_1206, symbol Device:LED_Small
- added R2: 330, Resistors_SMD:R_1206, symbol Device:R
- added U2: 74LV541, symbol speculatrix_ic:74LV541
- added U3: 74LV14, symbol speculatrix_ic:74LV14
- added U4: 74LV595, symbol speculatrix_ic:74LV595
- U1: symbol speculatrix_microcontroller:ATMEGA328PB -> SmartParallel-rescue:ATMEGA328PB-speculatrix_microcontroller
- renumbered C2 to C1, C1 to C2, C4 to C3, C5 to C4, C3 to C5, C9 to C6, C6 to C8, C8 to C9, D3 to D1, D7 to D10, D1 to D4, D8 to D5, D9 to D6, D5 to D7, D6 to D8, D4 to D9, P5 to P4, P6 to P5, R3 to R1, R11 to R10, R12 to R11, R13 to R12, R9 to R13, R10 to R14, R14 to R15, R1 to R18, R18 to R19, R6 to R3, R8 to R4, R2 to R5, R4 to R6, R5 to R7, R7 to R8, R15 to R9, SW2 to SW1
Connections:
- net Busy: now also U2.5 (A4)
- net Busy_buf: now also U2.15 (Y4)
- net D0: now also U4.15 (QA)
- net D1: now also U4.1 (QB)
- net D2: now also U4.2 (QC)
- net D3: now also U4.3 (QD)
- net D4: now also U4.4 (QE)
- net D5: now also U4.5 (QF)
- net D6: now also U4.6 (QG)
- net D7: now also U4.7 (QH)
- net GND: now also R2.2, U2.1 (~OE1), U2.10 (GND), U2.19 (~OE2), U3.7 (GND), U4.13 (~OE), U4.8 (GND)
- net PE: now also U2.3 (A2)
- net PE_buf: now also U2.17 (Y2)
- net SEL: now also U2.4 (A3), U3.3 (2A)
- net SER: now also U4.14 (SER)
- net SHCP: now also U4.11 (SHCP)
- net STCP: now also U4.12 (STCP)
- net Sel_buf: now also U2.16 (Y3)
- net VCC: now also D3.2 (A), U2.20 (VCC), U3.14 (VCC), U4.16 (VCC)
- net ~ACK: now also U2.2 (A1)
- net ~Ack_buf: now also U2.18 (Y1)
- net ~Autofeed: now also U2.9 (A8)
- net ~Autofeed_buf: now also U2.11 (Y8), U3.5 (3A)
- net ~Err_buf: now also U2.14 (Y5)
- net ~Error: now also U2.6 (A5), U3.1 (1A)
- net ~Init: now also U2.8 (A7)
- net ~Init_buf: now also U2.12 (Y7)
- net ~Strobe: now also U2.7 (A6)
- net ~Strobe_buf: now also U2.13 (Y6)
- net at R15.2: now also U4.10 (~MR)
- net at D7.2 (A): now also U3.2 (1Y)
- net at D8.2 (A): now also U3.4 (2Y)
- net at D9.2 (A): now also U3.6 (3Y)
- new net: D3.1 (K), R2.1
- no-connect marks 6 -> 8
Other:
- moved on the sheet: C2, C5, C9, D10, D7, D8, D9, J1, P2, P3, R16, R17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
